File: Hardware/Eagle Docs/TuringMixExpander.brd (EAGLE design)
At the start: 105 x 50.3 mm, 49 parts, among them IC1 TL074P, IC2 TL072P

Commit message: Gerbers manufactured OSHPark
Routing:
- net N$13: track 47.5 -> 41.0 mm
- net N$10: track 86.3 -> 81.5 mm
- net N$4: track 53.6 -> 49.5 mm
- net INPUT2: track 71.2 -> 68.0 mm
- net GND: track 250.0 -> 246.9 mm
- net INPUT4: track 104.7 -> 101.9 mm
- net INPUT1: track 52.6 -> 50.4 mm
- net N$17: track 21.0 -> 18.9 mm
- net INPUT3: track 89.7 -> 88.1 mm
- net N$11: track 77.0 -> 75.6 mm
- net N$12: track 53.0 -> 51.6 mm
- net N$27: track 48.7 -> 47.8 mm
- net N$7: track 88.2 -> 87.4 mm
- net SUMR: track 116.1 -> 115.4 mm
- net +12V: track 68.3 -> 67.7 mm
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
Commit message: Rev 3.1 Gerbers for OSH Park
Parts:
- added R13, R16: 10k, TomW:0207/7
- added R14, R15: 47k, TomW:0207/7
- moved U$1 39.5 mm to (80.0, 34.3), turned to 270 degrees
- moved R8 38.6 mm to (82.5, 44.5), turned to 90 degrees
- moved R7 36.5 mm to (82.5, 26.7), turned to 90 degrees
- moved R10 21.3 mm to (6.35, 15.2)
- moved C1 20.9 mm to (24.1, 6.35), turned to 90 degrees
- moved C2 20.7 mm to (21.6, 6.35), turned to 90 degrees
- moved R5 11.4 mm to (66.0, 20.3)
- moved R4 10.2 mm to (76.2, 17.8)
- moved U$3 9.16 mm to (8.89, 30.5), turned to 270 degrees
- moved R2 6.84 mm to (20.3, 15.2)
- moved OUT_LEFT 2.86 mm to (100.3, 25.1)
- moved OUT_LEFT1 2.86 mm to (88.9, 25.1)
- moved IC1 2.54 mm to (11.4, 6.35)
- moved IN_1A 2.54 mm to (66.0, 6.35)
- moved IN_2A 2.54 mm to (77.5, 6.35)
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Connections:
- net +12V: now also C1.1; no longer C1.2
- net GND: now also C1.2, R13.1, R16.1; no longer C1.1
- net N$10: now also R15.1, R16.2; no longer OUT_R.P$3, OUT_R1.P$3, R8.2
- net N$22: now also OUT_LEFT.P$3, OUT_LEFT1.P$3, R7.2; no longer OUT_LEFT.P$2, OUT_LEFT1.P$2
- net N$24: now also IC2.1, R15.2, R8.1; no longer OUT_R.P$2, OUT_R1.P$2
- net N$5: now also R14.2, R7.1; no longer R7.2
- net N$6: now also OUT_R.P$3, OUT_R1.P$3, R8.2; no longer IC2.1, R8.1
- net N$7: now also R13.2, R14.1; no longer OUT_LEFT.P$3, OUT_LEFT1.P$3, R7.1
Routing:
- net GND: track 246.9 -> 330.7 mm
- net N$7: track 87.4 -> 12.3 mm
- net N$10: track 81.5 -> 16.1 mm
- net N$23: track 83.2 -> 124.1 mm
- net N$5: track 4.23 -> 44.2 mm
- net GATE4: track 18.4 -> 57.5 mm
- net N$24: track 11.8 -> 49.5 mm, vias 0 -> 1
- net GATE2: track 35.4 -> 66.0 mm
- net GATE1: track 35.4 -> 61.7 mm, vias 0 -> 1
- net N$27: track 47.8 -> 29.3 mm
- net GATE3: track 18.5 -> 37.0 mm
- net N$6: track 3.81 -> 18.1 mm
- net N$3: track 51.1 -> 63.1 mm
- net N$1: track 92.2 -> 80.5 mm, vias 0 -> 1
- net N$28: track 8.98 -> 19.1 mm
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Other:
- board text added: "Turing Machine Expander 3 Vactrol Matrix Mixer Designed by Tom Whitwell In Herne Hill, London, March 2015 PCB Rev 3.1"
- board text removed: "Turing Machine Expander 3 Vactrol Matrix Mixer Designed by Tom Whitwell In Herne Hill, London, Feb 2015 PCB Rev 3"
