File: Hardware/Eagle Docs/TuringMixExpander.sch (EAGLE design)
At the start: 46 parts, among them IC1 TL074P, IC2 TL072P

Commit message: Rev 3.1 Gerbers for OSH Park
Parts:
- added R13, R16: 10k, TomW:R-EU_0207/7
- added R14, R15: 47k, TomW:R-EU_0207/7
Connections:
- net +12V: now also C1.1; no longer C1.2
- net GND: now also C1.2, R13.1, R16.1; no longer C1.1
- net N$10: now also R15.1, R16.2; no longer OUT_R.3, OUT_R1.3, R8.2
- net N$22: now also OUT_LEFT.3, OUT_LEFT1.3, R7.2; no longer OUT_LEFT.4, OUT_LEFT1.4
- net N$24: now also IC2A.OUT, R15.2, R8.1; no longer OUT_R.4, OUT_R1.4
- net N$5: now also R14.2, R7.1; no longer R7.2
- net N$6: now also OUT_R.3, OUT_R1.3, R8.2; no longer IC2A.OUT, R8.1
- net N$7: now also R13.2, R14.1; no longer OUT_LEFT.3, OUT_LEFT1.3, R7.1
Other:
- moved on the sheet: C1, IC2B, OUT_LEFT, OUT_LEFT1, OUT_R, R5, R7, R8
